Commit message: update

File: turtlebot_description/urdf/sensors/kinect.urdf.xacro (robot description, xacro)
@@ -30,10 +30,10 @@
         </geometry>
       </visual>
-  	  <collision>
+        <collision>
         <origin xyz="0.0 0.0 0.0" rpy="0 0 0"/>
-  	    <geometry>
-  	      <box size="0.07271 0.27794 0.073"/>
-  	    </geometry>
-  	  </collision>
+          <geometry>
+            <box size="0.07271 0.27794 0.073"/>
+          </geometry>
+        </collision>
       <inertial>
         <mass value="0.564" />
@@ -47,18 +47,18 @@
          files. However, for Gazebo simulation we need them, so we add them here.
          (Hence, don't publish them additionally!) -->
-	<joint name="camera_depth_joint" type="fixed">
-	  <origin xyz="0 ${2 * -kinect_cam_py} 0" rpy="0 0 0" />
-	  <parent link="camera_rgb_frame" />
-	  <child link="camera_depth_frame" />
-	</joint>
-	<link name="camera_depth_frame"/>
-	<joint name="camera_depth_optical_joint" type="fixed">
-	  <origin xyz="0 0 0" rpy="${-M_PI/2} 0 ${-M_PI/2}" />
-	  <parent link="camera_depth_frame" />
-	  <child link="camera_depth_optical_frame" />
-	</joint>
-	<link name="camera_depth_optical_frame"/>
-	<!-- Kinect sensor for simulation -->
-	<xacro:turtlebot_sim_3dsensor/>
+    <joint name="camera_depth_joint" type="fixed">
+      <origin xyz="0 ${2 * -kinect_cam_py} 0" rpy="0 0 0" />
+      <parent link="camera_rgb_frame" />
+      <child link="camera_depth_frame" />
+    </joint>
+    <link name="camera_depth_frame"/>
+    <joint name="camera_depth_optical_joint" type="fixed">
+      <origin xyz="0 0 0" rpy="${-M_PI/2} 0 ${-M_PI/2}" />
+      <parent link="camera_depth_frame" />
+      <child link="camera_depth_optical_frame" />
+    </joint>
+    <link name="camera_depth_optical_frame"/>
+    <!-- Kinect sensor for simulation -->
+    <xacro:turtlebot_sim_3dsensor/>
   </xacro:macro>
 </robot>

File: turtlebot_description/urdf/sensors/r200.urdf.xacro (robot description, xacro)
@@ -128,5 +128,5 @@
     </joint>
     <link name="camera_depth_optical_frame"/>
-  	<!-- Simulation sensor -->
+      <!-- Simulation sensor -->
     <xacro:turtlebot_sim_3dsensor/>
   </xacro:macro>

File: turtlebot_description/urdf/turtlebot_properties.urdf.xacro (robot description, xacro)
@@ -19,9 +19,9 @@
      (currently in development and awaiting feedback)
    -->
-	<xacro:property name="cam_px" value="-0.087" />
-<!--	<xacro:property name="cam_py" value="-0.0125" /> Y varies for different configurations. get sets in sensors_urdf -->
-	<xacro:property name="cam_pz" value="0.2870" />
-	<xacro:property name="cam_or" value="0" />
-	<xacro:property name="cam_op" value="0" />
-	<xacro:property name="cam_oy" value="0" />
+    <xacro:property name="cam_px" value="-0.087" />
+<!--    <xacro:property name="cam_py" value="-0.0125" /> Y varies for different configurations. get sets in sensors_urdf -->
+    <xacro:property name="cam_pz" value="0.2870" />
+    <xacro:property name="cam_or" value="0" />
+    <xacro:property name="cam_op" value="0" />
+    <xacro:property name="cam_oy" value="0" />
 </robot>
